Commit message: patvarkyti failai

File: src/dviratis_robotas/urdf/main.xacro (robot description, xacro)
@@ -1,12 +1,13 @@
 <?xml version="1.0"?>
-<robot name="dr_robotas" xmlns:xacro="http://www.ros.org/wiki/xacro">
-  <xacro:include filename="C:\ROS_ws\src\dr_robotas\model\colors.xacro" />
-  <xacro:include filename="C:\ROS_ws\src\dr_robotas\model\macros.xacro" />
-  <xacro:include filename="C:\ROS_ws\src\dr_robotas\model\param.xacro" />
+<robot name="dr_robotas"
+  xmlns:xacro="http://www.ros.org/wiki/xacro">
+  <xacro:include filename="$(find dviratis_robotas)/urdf/colors.xacro" />
+  <xacro:include filename="$(find dviratis_robotas)/urdf/macros.xacro" />
+  <xacro:include filename="$(find dviratis_robotas)/urdf/param.xacro" />
   <!-- links -->
   <link name="base_link">
     <visual name="base_link_visual">
       <geometry>
-          <box size="${total_length} ${total_width} ${base_z}" />
+        <box size="${total_length} ${total_width} ${base_z}" />
       </geometry>
       <origin xyz="${(total_length-pcb_x)/2+pcb_x_offset-base_padding} 0 0"/>
@@ -15,5 +16,5 @@
     <collision name="base_link_collision">
       <geometry>
-          <box size="${total_length} ${total_width} ${base_z}" />
+        <box size="${total_length} ${total_width} ${base_z}" />
       </geometry>
       <origin xyz="${(total_length-pcb_x)/2+pcb_x_offset-base_padding} 0 0"/>
@@ -33,22 +34,22 @@
   <link name="caster_front_link">
     <visual name='caster_visual'>
-        <geometry>
-            <sphere radius="${caster_wheel_r}"/>
-        </geometry>
+      <geometry>
+        <sphere radius="${caster_wheel_r}"/>
+      </geometry>
     </visual>
     <collision name='caster_collision'>
-        <geometry>
-            <sphere radius="${caster_wheel_r}"/>
-        </geometry>
-        <surface>
-            <friction>
-                <ode>
-                    <mu>0</mu>
-                    <mu2>0</mu2>
-                    <slip1>1.0</slip1>
-                    <slip2>1.0</slip2>
-                </ode>
-            </friction>
-        </surface>
+      <geometry>
+        <sphere radius="${caster_wheel_r}"/>
+      </geometry>
+      <surface>
+        <friction>
+          <ode>
+            <mu>0</mu>
+            <mu2>0</mu2>
+            <slip1>1.0</slip1>
+            <slip2>1.0</slip2>
+          </ode>
+        </friction>
+      </surface>
     </collision>
   </link>

File: src/dviratis_robotas/urdf/param.xacro (robot description, xacro)
@@ -4,10 +4,10 @@
     <xacro:property name="wheel_w" value="0.026" />
     <xacro:property name="wheel_m" value="0.026" />
-	<xacro:property name="rpy_x" value="0.1" />
-	<xacro:property name="rpy_y" value="0.07" />
-	<xacro:property name="rpy_z" value="0.035" />
-	<xacro:property name="batt_x" value="0.12" />
-	<xacro:property name="batt_y" value="0.03" />
-	<xacro:property name="batt_z" value="0.04" />
+    <xacro:property name="rpy_x" value="0.1" />
+    <xacro:property name="rpy_y" value="0.07" />
+    <xacro:property name="rpy_z" value="0.035" />
+    <xacro:property name="batt_x" value="0.12" />
+    <xacro:property name="batt_y" value="0.03" />
+    <xacro:property name="batt_z" value="0.04" />
     <xacro:property name="base_z" value="0.005" />
     <xacro:property name="pcb_x" value="0.05" />

Commit message: Testavimas kontroleriui (bet greiciausiai ne to reikia)

File: src/dviratis_robotas/urdf/main.xacro (robot description, xacro)
@@ -2,7 +2,5 @@
 <robot name="dr_robotas"
   xmlns:xacro="http://www.ros.org/wiki/xacro">
-  <xacro:include filename="$(find dviratis_robotas)/urdf/colors.xacro" />
   <xacro:include filename="$(find dviratis_robotas)/urdf/macros.xacro" />
-  <xacro:include filename="$(find dviratis_robotas)/urdf/param.xacro" />
   <!-- links -->
   <link name="base_link">
@@ -79,3 +77,27 @@
     <joint_properties damping="1.0" friction="1.0"/>
   </joint>
+  <transmission name="left_wheel_transmission">
+    <type>transmission_interface/SimpleTransmission</type>
+    <joint name="base_to_lwheel">
+      <hardwareInterface>hardware_interface/VelocityJointInterface</hardwareInterface>
+    </joint>
+    <actuator name="left_wheel_actuator">
+      <mechanicalReduction>7</mechanicalReduction>
+      <hardwareInterface>hardware_interface/VelocityJointInterface</hardwareInterface>
+    </actuator>
+  </transmission>
+  <transmission name="right_wheel_transmission">
+    <type>transmission_interface/SimpleTransmission</type>
+    <joint name="base_to_rwheel">
+      <hardwareInterface>hardware_interface/VelocityJointInterface</hardwareInterface>
+    </joint>
+    <actuator name="right_wheel_actuator">
+      <mechanicalReduction>7</mechanicalReduction>
+      <hardwareInterface>hardware_interface/VelocityJointInterface</hardwareInterface>
+    </actuator>
+  </transmission>
+  <gazebo>
+    <plugin name="gazebo_ros_control" filename="libgazebo_ros_contol.so">
+    </plugin>
+  </gazebo>
 </robot>
