Commit message: veikia rviz, neveikia gazebo

File: src/dviratis_robotas/urdf/macros.xacro (robot description, xacro)
@@ -53,5 +53,5 @@
 		</joint>
 		<joint name="base_to_batt" type="fixed">
-			<parent link="base_link"/>
+			<parent link="chassis_link"/>
 			<child link="${name}_batt"/>
 			<origin xyz="${x} ${y+batt_y/2-(batt_y+rpy_y)/2} ${z}"/>

File: src/dviratis_robotas/urdf/main.xacro (robot description, xacro)
@@ -3,7 +3,8 @@
   xmlns:xacro="http://www.ros.org/wiki/xacro">
   <xacro:include filename="$(find dviratis_robotas)/urdf/macros.xacro" />
+  <xacro:include filename="$(find dviratis_robotas)/urdf/gazebo.gazebo" />
   <!-- links -->
-  <link name="base_link">
-    <visual name="base_link_visual">
+  <link name="chassis_link">
+    <visual name="chassis_link_visual">
       <geometry>
         <box size="${total_length} ${total_width} ${base_z}" />
@@ -12,5 +13,5 @@
       <material name="orange"/>
     </visual>
-    <collision name="base_link_collision">
+    <collision name="chassis_link_collision">
       <geometry>
         <box size="${total_length} ${total_width} ${base_z}" />
@@ -27,5 +28,5 @@
     </visual>
   </link>
-  <xacro:battery_and_rpy name="link_right_wheel" x="${gap_pcb_bat+(batt_x+pcb_x)/2+pcb_x_offset}" y="${0}" z="${(batt_z+base_z)/2}"/>
+  <xacro:battery_and_rpy name="link_blokas" x="${gap_pcb_bat+(batt_x+pcb_x)/2+pcb_x_offset}" y="${0}" z="${(batt_z+base_z)/2}"/>
   <xacro:wheel_link name="right_wheel_link"/>
   <xacro:wheel_link name="left_wheel_link"/>
@@ -54,15 +55,15 @@
   <!-- joints -->
   <joint name="base_to_caster" type="fixed">
-    <parent link="base_link"/>
+    <parent link="chassis_link"/>
     <child link="caster_front_link"/>
     <origin xyz="${(total_length-pcb_x)+pcb_x_offset-base_padding} 0 -${caster_wheel_r+pcb_z/2}"/>
   </joint>
   <joint name="base_to_pcb" type="fixed">
-    <parent link="base_link"/>
+    <parent link="chassis_link"/>
     <child link="pcb"/>
     <origin xyz="${pcb_x_offset} 0 ${pcb_z/2+base_z/2}"/>
   </joint>
   <joint name="base_to_rwheel" type="continuous">
-    <parent link="base_link"/>
+    <parent link="chassis_link"/>
     <child link="right_wheel_link"/>
     <origin xyz="0 ${-(wheel_w+total_width)/2} -${motor_r+pcb_z/2}"/>
@@ -71,5 +72,5 @@
   </joint>
   <joint name="base_to_lwheel" type="continuous">
-    <parent link="base_link"/>
+    <parent link="chassis_link"/>
     <child link="left_wheel_link"/>
     <origin xyz="0 ${(wheel_w+total_width)/2} -${motor_r+pcb_z/2}"/>
@@ -77,27 +78,11 @@
     <joint_properties damping="1.0" friction="1.0"/>
   </joint>
-  <transmission name="left_wheel_transmission">
-    <type>transmission_interface/SimpleTransmission</type>
-    <joint name="base_to_lwheel">
-      <hardwareInterface>hardware_interface/VelocityJointInterface</hardwareInterface>
-    </joint>
-    <actuator name="left_wheel_actuator">
-      <mechanicalReduction>7</mechanicalReduction>
-      <hardwareInterface>hardware_interface/VelocityJointInterface</hardwareInterface>
-    </actuator>
-  </transmission>
-  <transmission name="right_wheel_transmission">
-    <type>transmission_interface/SimpleTransmission</type>
-    <joint name="base_to_rwheel">
-      <hardwareInterface>hardware_interface/VelocityJointInterface</hardwareInterface>
-    </joint>
-    <actuator name="right_wheel_actuator">
-      <mechanicalReduction>7</mechanicalReduction>
-      <hardwareInterface>hardware_interface/VelocityJointInterface</hardwareInterface>
-    </actuator>
-  </transmission>
-  <gazebo>
-    <plugin name="gazebo_ros_control" filename="libgazebo_ros_contol.so">
-    </plugin>
-  </gazebo>
+  <!-- Create a dummy link as base link -->
+  <link name='base_link'>
+    <pose>0 0 0 0 0 0</pose>
+  </link>
+  <joint type="fixed" name="base_link_to_chassis">
+    <child link="chassis_link"/>
+    <parent link="base_link"/>
+  </joint>
 </robot>
