Commit message: Issprestos problemos su gazeboo modeliu (#1)
* Veikia simuliatorius

* Paderintos vertes

* atsisakyta savos rasybos modelio del klaidu, jo vietoj idetas kitas

* Patvarkyti matmenys

File: src/dviratis_robotas/urdf/dr_robotas.xacro (robot description, xacro)
@@ -1,88 +1,141 @@
-<?xml version="1.0"?>
+<?xml version='1.0'?>
+<!-- choose a name space and start xacro -->
 <robot name="dr_robotas"
-  xmlns:xacro="http://www.ros.org/wiki/xacro">
-  <xacro:include filename="$(find dviratis_robotas)/urdf/macros.xacro" />
-  <xacro:include filename="$(find dviratis_robotas)/urdf/gazebo.gazebo" />
-  <!-- links -->
-  <link name="chassis_link">
-    <visual name="chassis_link_visual">
-      <geometry>
-        <box size="${total_length} ${total_width} ${base_z}" />
-      </geometry>
-      <origin xyz="${(total_length-pcb_x)/2+pcb_x_offset-base_padding} 0 0"/>
-      <material name="orange"/>
-    </visual>
-    <collision name="chassis_link_collision">
-      <geometry>
-        <box size="${total_length} ${total_width} ${base_z}" />
-      </geometry>
-      <origin xyz="${(total_length-pcb_x)/2+pcb_x_offset-base_padding} 0 0"/>
-    </collision>
-  </link>
-  <link name="pcb">
-    <visual>
-      <geometry>
-        <box size="${pcb_x} ${pcb_y} ${pcb_z}" />
-      </geometry>
-      <material name="green"/>
-    </visual>
-  </link>
-  <xacro:battery_and_rpy name="link_blokas" x="${gap_pcb_bat+(batt_x+pcb_x)/2+pcb_x_offset}" y="${0}" z="${(batt_z+base_z)/2}"/>
-  <xacro:wheel_link name="right_wheel_link"/>
-  <xacro:wheel_link name="left_wheel_link"/>
-  <link name="caster_front_link">
-    <visual name='caster_visual'>
-      <geometry>
-        <sphere radius="${caster_wheel_r}"/>
-      </geometry>
-    </visual>
-    <collision name='caster_collision'>
-      <geometry>
-        <sphere radius="${caster_wheel_r}"/>
-      </geometry>
-      <surface>
-        <friction>
-          <ode>
-            <mu>0</mu>
-            <mu2>0</mu2>
-            <slip1>1.0</slip1>
-            <slip2>1.0</slip2>
-          </ode>
-        </friction>
-      </surface>
-    </collision>
-  </link>
-  <!-- joints -->
-  <joint name="base_to_caster" type="fixed">
-    <parent link="chassis_link"/>
-    <child link="caster_front_link"/>
-    <origin xyz="${(total_length-pcb_x)+pcb_x_offset-base_padding} 0 -${caster_wheel_r+pcb_z/2}"/>
-  </joint>
-  <joint name="base_to_pcb" type="fixed">
-    <parent link="chassis_link"/>
-    <child link="pcb"/>
-    <origin xyz="${pcb_x_offset} 0 ${pcb_z/2+base_z/2}"/>
-  </joint>
-  <joint name="base_to_rwheel" type="continuous">
-    <parent link="chassis_link"/>
-    <child link="right_wheel_link"/>
-    <origin xyz="0 ${-(wheel_w+total_width)/2} -${motor_r+pcb_z/2}"/>
-    <limit effort="10000" velocity="1000"/>
-    <joint_properties damping="1.0" friction="1.0"/>
-  </joint>
-  <joint name="base_to_lwheel" type="continuous">
-    <parent link="chassis_link"/>
-    <child link="left_wheel_link"/>
-    <origin xyz="0 ${(wheel_w+total_width)/2} -${motor_r+pcb_z/2}"/>
-    <limit effort="10000" velocity="1000"/>
-    <joint_properties damping="1.0" friction="1.0"/>
-  </joint>
-  <!-- Create a dummy link as base link -->
-  <link name='base_link'>
-    <pose>0 0 0 0 0 0</pose>
-  </link>
-  <joint type="fixed" name="base_link_to_chassis">
-    <child link="chassis_link"/>
-    <parent link="base_link"/>
-  </joint>
+    xmlns:xacro="http://www.ros.org/wiki/xacro">
+    <!-- Start by including all required xacro files which hold the macros -->
+    <xacro:include filename="$(find dviratis_robotas)/urdf/diff_drive.gazebo" />
+    <xacro:include filename="$(find dviratis_robotas)/urdf/materials.xacro" />
+    <xacro:include filename="$(find dviratis_robotas)/urdf/macros.xacro" />
+    <xacro:include filename="$(find dviratis_robotas)/urdf/parameter.xacro" />
+    <!-- Create a dummy link as base link -->
+    <link name='base_link'>
+        <pose>0 0 0 0 0 0</pose>
+    </link>
+    <joint type="fixed" name="base_link_to_chassis">
+        <child link="chassis_link"/>
+        <parent link="base_link"/>
+    </joint>
+    <!-- Define the chassis of the differential drive robot, which is our base -->
+    <link name='chassis_link'>
+        <!-- Define inertial system for the chassis -->
+        <inertial>
+            <mass value="${m_chassis}"/>
+            <xacro:box_inertia m="${m_chassis}" x="${x_chassis}" y="${y_chassis}" z="${z_chassis}"/>
+        </inertial>
+        <!-- Define collision sorrounding box -->
+        <collision name='collision'>
+            <origin xyz="0 0 0" rpy=" 0 0 0"/>
+            <geometry>
+                <box size="${x_chassis} ${y_chassis} ${z_chassis}"/>
+            </geometry>
+        </collision>
+        <!-- Define visualization structure -->
+        <visual name='base_link_visual'>
+            <origin xyz="0 0 0" rpy=" 0 0 0"/>
+            <geometry>
+                <box size="${x_chassis} ${y_chassis} ${z_chassis}"/>
+            </geometry>
+        </visual>
+        <!-- Add the caster wheel! Here we simply assume complete slippage, thus we do not require that it rotates! -->
+        <collision name='caster_collision'>
+            <origin xyz="${-(r_wheel/2)+x_chassis/2} 0 ${-r_wheel/2-z_chassis/2}" rpy=" 0 0 0"/>
+            <geometry>
+                <sphere radius="${r_wheel/2}"/>
+            </geometry>
+            <surface>
+                <friction>
+                    <ode>
+                        <mu>0</mu>
+                        <mu2>0</mu2>
+                        <slip1>1.0</slip1>
+                        <slip2>1.0</slip2>
+                    </ode>
+                </friction>
+            </surface>
+        </collision>
+        <visual name='caster_visual'>
+            <origin xyz="${-(r_wheel/2)+x_chassis/2} 0 ${-r_wheel/2-z_chassis/2}" rpy=" 0 0 0"/>
+            <geometry>
+                <sphere radius="${r_wheel/2}"/>
+            </geometry>
+        </visual>
+    </link>
+    <!-- Add the wheels for the robot -->
+    <link name="left_wheel">
+        <collision name="collision">
+            <origin xyz="0 0 0" rpy="0 1.5707 1.5707"/>
+            <geometry>
+                <cylinder radius="${r_wheel}" length="${h_wheel}"/>
+            </geometry>
+            <surface>
+                <friction>
+                    <ode>
+                        <mu>1.0</mu>
+                        <mu2>1.0</mu2>
+                        <slip1>0.0</slip1>
+                        <slip2>0.0</slip2>
+                    </ode>
+                </friction>
+            </surface>
+        </collision>
+        <visual name="left_wheel_visual">
+            <origin xyz="0 0 0" rpy="0 1.5707 1.5707"/>
+            <geometry>
+                <cylinder radius="${r_wheel}" length="${h_wheel}"/>
+            </geometry>
+        </visual>
+        <inertial>
+            <origin xyz="0 0 0" rpy="0 1.5707 1.5707"/>
+            <mass value="${m_wheel}"/>
+            <cylinder_inertia m="${m_wheel}" r="${r_wheel}" h="${h_wheel}"/>
+            <xacro:cylinder_inertia m="${m_wheel}" r="${r_wheel}" h="${h_wheel}"/>
+        </inertial>
+    </link>
+    <link name="right_wheel">
+        <collision name="collision">
+            <origin xyz="0 0 0" rpy="0 1.5707 1.5707"/>
+            <geometry>
+                <cylinder radius="${r_wheel}" length="${h_wheel}"/>
+            </geometry>
+            <surface>
+                <friction>
+                    <ode>
+                        <mu>1.0</mu>
+                        <mu2>1.0</mu2>
+                        <slip1>0.0</slip1>
+                        <slip2>0.0</slip2>
+                    </ode>
+                </friction>
+            </surface>
+        </collision>
+        <visual name="right_wheel_visual">
+            <origin xyz="0 0 0" rpy="0 1.5707 1.5707"/>
+            <geometry>
+                <cylinder radius="${r_wheel}" length="${h_wheel}"/>
+            </geometry>
+        </visual>
+        <inertial>
+            <origin xyz="0 0 0" rpy="0 1.5707 1.5707"/>
+            <mass value="${m_wheel}"/>
+            <cylinder_inertia m="${m_wheel}" r="${r_wheel}" h="${h_wheel}"/>
+            <xacro:cylinder_inertia m="${m_wheel}" r="${r_wheel}" h="${h_wheel}"/>
+        </inertial>
+    </link>
+    <!-- Set joints for the wheels which can be controlled over ROS -->
+    <joint type="continuous" name="left_wheel_hinge">
+        <origin xyz="${-x_chassis/4} ${y_chassis/2+h_wheel/2} ${-z_chassis/2}" rpy="0 0 0"/>
+        <child link="left_wheel"/>
+        <parent link="base_link"/>
+        <axis xyz="0 1 0" rpy="0 0 0"/>
+        <limit effort="100" velocity="100"/>
+        <joint_properties damping="0.0" friction="0.0"/>
+    </joint>
+    <joint type="continuous" name="right_wheel_hinge">
+        <origin xyz="${-x_chassis/4} ${-y_chassis/2-h_wheel/2} ${-z_chassis/2}" rpy="0 0 0"/>
+        <child link="right_wheel"/>
+        <parent link="base_link"/>
+        <axis xyz="0 1 0" rpy="0 0 0"/>
+        <limit effort="100" velocity="100"/>
+        <joint_properties damping="0.0" friction="0.0"/>
+    </joint>
 </robot>

File: src/dviratis_robotas/urdf/macros.xacro (robot description, xacro)
@@ -1,60 +1,9 @@
 <?xml version="1.0"?>
 <robot xmlns:xacro="http://www.ros.org/wiki/xacro">
-	<xacro:include filename="$(find dviratis_robotas)/urdf/colors.xacro" />
-	<xacro:include filename="$(find dviratis_robotas)/urdf/param.xacro" />
-	<xacro:macro name="box_inertia" params="m x y z">
-		<inertia ixx="${m*(y*y+z*z)/12}" ixy = "0" ixz = "0" iyy="${m*(x*x+z*z)/12}" iyz = "0" izz="${m*(x*x+z*z)/12}" />
-	</xacro:macro>
-	<xacro:macro name="cylinder_inertia" params="m r h">
-		<inertia ixx="${m*(3*r*r+h*h)/12}" ixy = "0" ixz = "0" iyy="${m*(3*r*r+h*h)/12}" iyz = "0" izz="${m*r*r/2}" />
-	</xacro:macro>
-	<macro name="wheel_link" params="name">
-		<link name="${name}">
-			<inertial>
-				<mass value="${wheel_m}"/>
-				<origin rpy="0 1.5707 1.5707" xyz="0 0 0"/>
-				<cylinder_inertia m="${wheel_m}" r="${wheel_r}" h="${wheel_w}"/>
-			</inertial>
-			<collision name="${name}_collision">
-				<origin rpy="0 1.5707 1.5707" xyz="0 0 0"/>
-				<geometry>
-					<cylinder length="${wheel_m}" radius="${wheel_r}"/>
-				</geometry>
-			</collision>
-			<visual name="${name}_visual">
-				<origin rpy="0 1.5707 1.5707" xyz="0 0 0"/>
-				<geometry>
-					<cylinder length="${wheel_m}" radius="${wheel_r}"/>
-				</geometry>
-			</visual>
-		</link>
-	</macro>
-	<macro name="battery_and_rpy" params="name x y z">
-		<link name="${name}_rpy">
-			<visual>
-				<geometry>
-					<box size="${rpy_x} ${rpy_y} ${rpy_z}" />
-				</geometry>
-				<material name="red"/>
-			</visual>
-		</link>
-		<link name="${name}_batt">
-			<visual>
-				<geometry>
-					<box size="${batt_x} ${batt_y} ${batt_z}" />
-				</geometry>
-				<material name="yellow"/>
-			</visual>
-		</link>
-		<joint name="batt_to_rpy" type="fixed">
-			<parent link="${name}_batt"/>
-			<child link="${name}_rpy"/>
-			<origin xyz="0 ${(rpy_y+batt_y)/2} ${(-batt_z+rpy_z)/2}"/>
-		</joint>
-		<joint name="base_to_batt" type="fixed">
-			<parent link="chassis_link"/>
-			<child link="${name}_batt"/>
-			<origin xyz="${x} ${y+batt_y/2-(batt_y+rpy_y)/2} ${z}"/>
-		</joint>
-	</macro>
+    <xacro:macro name="box_inertia" params="m x y z">
+        <inertia ixx="${m*(y*y+z*z)/12}" ixy = "0" ixz = "0" iyy="${m*(x*x+z*z)/12}" iyz = "0" izz="${m*(x*x+z*z)/12}" />
+    </xacro:macro>
+    <xacro:macro name="cylinder_inertia" params="m r h">
+        <inertia ixx="${m*(3*r*r+h*h)/12}" ixy = "0" ixz = "0" iyy="${m*(3*r*r+h*h)/12}" iyz = "0" izz="${m*r*r/2}" />
+    </xacro:macro>
 </robot>

File: src/dviratis_robotas/urdf/parameter.xacro (robot description, xacro)
@@ -3,14 +3,14 @@
     <!-- Define parameter for the differential drive robot -->
     <!-- Parameter for the chassis, size [m] and mass [kg] -->
-    <xacro:property name="x_chassis" value="0.5" />
-    <xacro:property name="y_chassis" value="0.3" />
-    <xacro:property name="z_chassis" value="0.15" />
-    <xacro:property name="m_chassis" value="10.0" />
+    <xacro:property name="x_chassis" value="0.23" />
+    <xacro:property name="y_chassis" value="0.12" />
+    <xacro:property name="z_chassis" value="0.01" />
+    <xacro:property name="m_chassis" value="1.0" />
     <!-- Parameter for the wheels, radius [m], height [m], mass [kg], torque [Nm], wheelbase [m] -->
-    <xacro:property name="r_wheel" value="0.1075"/>
-    <xacro:property name="h_wheel" value="0.03" />
-    <xacro:property name="m_wheel" value="3.0" />
+    <xacro:property name="r_wheel" value="0.035"/>
+    <xacro:property name="h_wheel" value="0.025" />
+    <xacro:property name="m_wheel" value="0.03" />
     <xacro:property name="torque_wheel" value="10" />
-    <xacro:property name="L_wheel" value="0.1788" />
+    <xacro:property name="L_wheel" value="0.00" />
     <!-- Parameters for the Hukoyu Laser -->
     <xacro:property name="x_hokuyo" value="0.1" />

File: src/dviratis_robotas/urdf_old/param.xacro (robot description, xacro)
@@ -3,5 +3,5 @@
     <xacro:property name="wheel_r" value="0.034" />
     <xacro:property name="wheel_w" value="0.026" />
-    <xacro:property name="wheel_m" value="0.026" />
+    <xacro:property name="wheel_m" value="3.0" />
     <xacro:property name="rpy_x" value="0.1" />
     <xacro:property name="rpy_y" value="0.07" />

Commit message: RPY ir baterijos blokas

File: src/dviratis_robotas/urdf/dr_robotas.xacro (robot description, xacro)
@@ -36,4 +36,29 @@
                 <box size="${x_chassis} ${y_chassis} ${z_chassis}"/>
             </geometry>
+            <material name="yellow"/>
+        </visual>
+        <!-- RPY and batt block -->
+        <visual name='batt_rpy_collision'>
+            <origin xyz="${-0.03} 0 ${0.02+z_chassis/2}" rpy=" 0 0 0"/>
+            <geometry>
+                <box size="${0.12} ${0.1} ${0.04}" />
+            </geometry>
+            <surface>
+                <friction>
+                    <ode>
+                        <mu>0</mu>
+                        <mu2>0</mu2>
+                        <slip1>1.0</slip1>
+                        <slip2>1.0</slip2>
+                    </ode>
+                </friction>
+            </surface>
+        </visual>
+        <visual name='batt_rpy_visual'>
+            <origin xyz="${-0.03} 0 ${0.02+z_chassis/2}" rpy=" 0 0 0"/>
+            <geometry>
+                <box size="${0.12} ${0.1} ${0.04}" />
+            </geometry>
+            <material name="white"/>
         </visual>
         <!-- Add the caster wheel! Here we simply assume complete slippage, thus we do not require that it rotates! -->
@@ -59,4 +84,5 @@
                 <sphere radius="${r_wheel/2}"/>
             </geometry>
+            <material name="black"/>
         </visual>
     </link>
@@ -84,4 +110,5 @@
                 <cylinder radius="${r_wheel}" length="${h_wheel}"/>
             </geometry>
+            <material name="black"/>
         </visual>
         <inertial>
@@ -114,4 +141,5 @@
                 <cylinder radius="${r_wheel}" length="${h_wheel}"/>
             </geometry>
+            <material name="black"/>
         </visual>
         <inertial>

File: src/dviratis_robotas/urdf/parameter.xacro (robot description, xacro)
@@ -13,4 +13,11 @@
     <xacro:property name="torque_wheel" value="10" />
     <xacro:property name="L_wheel" value="0.00" />
+    <!-- Camera parameters -->
+    <xacro:property name="r_camera" value="0.1" />
+    <xacro:property name="h_camera" value="0.1" />
+    <!-- Radar parameters -->
+    <xacro:property name="x_radar" value="0.1" />
+    <xacro:property name="y_radar" value="0.1" />
+    <xacro:property name="z_radar" value="0.1" />
     <!-- Parameters for the Hukoyu Laser -->
     <xacro:property name="x_hokuyo" value="0.1" />

Commit message: Pafixintas collision ir visual rpy_batt blokui

File: src/dviratis_robotas/urdf/dr_robotas.xacro (robot description, xacro)
@@ -39,5 +39,5 @@
         </visual>
         <!-- RPY and batt block -->
-        <visual name='batt_rpy_collision'>
+        <collision name='batt_rpy_collision'>
             <origin xyz="${-0.03} 0 ${0.02+z_chassis/2}" rpy=" 0 0 0"/>
             <geometry>
@@ -54,5 +54,5 @@
                 </friction>
             </surface>
-        </visual>
+        </collision>
         <visual name='batt_rpy_visual'>
             <origin xyz="${-0.03} 0 ${0.02+z_chassis/2}" rpy=" 0 0 0"/>
@@ -60,5 +60,7 @@
                 <box size="${0.12} ${0.1} ${0.04}" />
             </geometry>
-            <material name="white"/>
+            <material name="red">
+                <color rgba="0.80078125 0.12890625 0.1328125 1.0"/>
+            </material>
         </visual>
         <!-- Add the caster wheel! Here we simply assume complete slippage, thus we do not require that it rotates! -->
