Commit message: Uzdetas radaro pcb

File: src/dviratis_robotas/urdf/dr_robotas.xacro (robot description, xacro)
@@ -2,170 +2,184 @@
 <!-- choose a name space and start xacro -->
 <robot name="dr_robotas"
-    xmlns:xacro="http://www.ros.org/wiki/xacro">
-    <!-- Start by including all required xacro files which hold the macros -->
-    <xacro:include filename="$(find dviratis_robotas)/urdf/diff_drive.gazebo" />
-    <xacro:include filename="$(find dviratis_robotas)/urdf/materials.xacro" />
-    <xacro:include filename="$(find dviratis_robotas)/urdf/macros.xacro" />
-    <xacro:include filename="$(find dviratis_robotas)/urdf/parameter.xacro" />
-    <!-- Create a dummy link as base link -->
-    <link name='base_link'>
-        <pose>0 0 0 0 0 0</pose>
-    </link>
-    <joint type="fixed" name="base_link_to_chassis">
-        <child link="chassis_link"/>
-        <parent link="base_link"/>
-    </joint>
-    <!-- Define the chassis of the differential drive robot, which is our base -->
-    <link name='chassis_link'>
-        <!-- Define inertial system for the chassis -->
-        <inertial>
-            <mass value="${m_chassis}"/>
-            <xacro:box_inertia m="${m_chassis}" x="${x_chassis}" y="${y_chassis}" z="${z_chassis}"/>
-        </inertial>
-        <!-- Define collision sorrounding box -->
-        <collision name='collision'>
-            <origin xyz="0 0 0" rpy=" 0 0 0"/>
-            <geometry>
-                <box size="${x_chassis} ${y_chassis} ${z_chassis}"/>
-            </geometry>
-        </collision>
-        <!-- Define visualization structure -->
-        <visual name='base_link_visual'>
-            <origin xyz="0 0 0" rpy=" 0 0 0"/>
-            <geometry>
-                <box size="${x_chassis} ${y_chassis} ${z_chassis}"/>
-            </geometry>
-            <material name="yellow"/>
-        </visual>
-        <!-- RPY and batt block -->
-        <collision name='batt_rpy_collision'>
-            <origin xyz="${-0.03} 0 ${0.02+z_chassis/2}" rpy=" 0 0 0"/>
-            <geometry>
-                <box size="${0.12} ${0.1} ${0.04}" />
-            </geometry>
-            <surface>
-                <friction>
-                    <ode>
-                        <mu>0</mu>
-                        <mu2>0</mu2>
-                        <slip1>1.0</slip1>
-                        <slip2>1.0</slip2>
-                    </ode>
-                </friction>
-            </surface>
-        </collision>
-        <visual name='batt_rpy_visual'>
-            <origin xyz="${-0.03} 0 ${0.02+z_chassis/2}" rpy=" 0 0 0"/>
-            <geometry>
-                <box size="${0.12} ${0.1} ${0.04}" />
-            </geometry>
-            <material name="red">
-                <color rgba="0.80078125 0.12890625 0.1328125 1.0"/>
-            </material>
-        </visual>
-        <!-- Add the caster wheel! Here we simply assume complete slippage, thus we do not require that it rotates! -->
-        <collision name='caster_collision'>
-            <origin xyz="${-(r_wheel/2)+x_chassis/2} 0 ${-r_wheel/2-z_chassis/2}" rpy=" 0 0 0"/>
-            <geometry>
-                <sphere radius="${r_wheel/2}"/>
-            </geometry>
-            <surface>
-                <friction>
-                    <ode>
-                        <mu>0</mu>
-                        <mu2>0</mu2>
-                        <slip1>1.0</slip1>
-                        <slip2>1.0</slip2>
-                    </ode>
-                </friction>
-            </surface>
-        </collision>
-        <visual name='caster_visual'>
-            <origin xyz="${-(r_wheel/2)+x_chassis/2} 0 ${-r_wheel/2-z_chassis/2}" rpy=" 0 0 0"/>
-            <geometry>
-                <sphere radius="${r_wheel/2}"/>
-            </geometry>
-            <material name="black"/>
-        </visual>
-    </link>
-    <!-- Add the wheels for the robot -->
-    <link name="left_wheel">
-        <collision name="collision">
-            <origin xyz="0 0 0" rpy="0 1.5707 1.5707"/>
-            <geometry>
-                <cylinder radius="${r_wheel}" length="${h_wheel}"/>
-            </geometry>
-            <surface>
-                <friction>
-                    <ode>
-                        <mu>1.0</mu>
-                        <mu2>1.0</mu2>
-                        <slip1>0.0</slip1>
-                        <slip2>0.0</slip2>
-                    </ode>
-                </friction>
-            </surface>
-        </collision>
-        <visual name="left_wheel_visual">
-            <origin xyz="0 0 0" rpy="0 1.5707 1.5707"/>
-            <geometry>
-                <cylinder radius="${r_wheel}" length="${h_wheel}"/>
-            </geometry>
-            <material name="black"/>
-        </visual>
-        <inertial>
-            <origin xyz="0 0 0" rpy="0 1.5707 1.5707"/>
-            <mass value="${m_wheel}"/>
-            <cylinder_inertia m="${m_wheel}" r="${r_wheel}" h="${h_wheel}"/>
-            <xacro:cylinder_inertia m="${m_wheel}" r="${r_wheel}" h="${h_wheel}"/>
-        </inertial>
-    </link>
-    <link name="right_wheel">
-        <collision name="collision">
-            <origin xyz="0 0 0" rpy="0 1.5707 1.5707"/>
-            <geometry>
-                <cylinder radius="${r_wheel}" length="${h_wheel}"/>
-            </geometry>
-            <surface>
-                <friction>
-                    <ode>
-                        <mu>1.0</mu>
-                        <mu2>1.0</mu2>
-                        <slip1>0.0</slip1>
-                        <slip2>0.0</slip2>
-                    </ode>
-                </friction>
-            </surface>
-        </collision>
-        <visual name="right_wheel_visual">
-            <origin xyz="0 0 0" rpy="0 1.5707 1.5707"/>
-            <geometry>
-                <cylinder radius="${r_wheel}" length="${h_wheel}"/>
-            </geometry>
-            <material name="black"/>
-        </visual>
-        <inertial>
-            <origin xyz="0 0 0" rpy="0 1.5707 1.5707"/>
-            <mass value="${m_wheel}"/>
-            <cylinder_inertia m="${m_wheel}" r="${r_wheel}" h="${h_wheel}"/>
-            <xacro:cylinder_inertia m="${m_wheel}" r="${r_wheel}" h="${h_wheel}"/>
-        </inertial>
-    </link>
-    <!-- Set joints for the wheels which can be controlled over ROS -->
-    <joint type="continuous" name="left_wheel_hinge">
-        <origin xyz="${-x_chassis/4} ${y_chassis/2+h_wheel/2} ${-z_chassis/2}" rpy="0 0 0"/>
-        <child link="left_wheel"/>
-        <parent link="base_link"/>
-        <axis xyz="0 1 0" rpy="0 0 0"/>
-        <limit effort="100" velocity="100"/>
-        <joint_properties damping="0.0" friction="0.0"/>
-    </joint>
-    <joint type="continuous" name="right_wheel_hinge">
-        <origin xyz="${-x_chassis/4} ${-y_chassis/2-h_wheel/2} ${-z_chassis/2}" rpy="0 0 0"/>
-        <child link="right_wheel"/>
-        <parent link="base_link"/>
-        <axis xyz="0 1 0" rpy="0 0 0"/>
-        <limit effort="100" velocity="100"/>
-        <joint_properties damping="0.0" friction="0.0"/>
-    </joint>
+	xmlns:xacro="http://www.ros.org/wiki/xacro">
+	<!-- Start by including all required xacro files which hold the macros -->
+	<xacro:include filename="$(find dviratis_robotas)/urdf/diff_drive.gazebo" />
+	<xacro:include filename="$(find dviratis_robotas)/urdf/materials.xacro" />
+	<xacro:include filename="$(find dviratis_robotas)/urdf/macros.xacro" />
+	<xacro:include filename="$(find dviratis_robotas)/urdf/parameter.xacro" />
+	<!-- Create a dummy link as base link -->
+	<link name='base_link'>
+		<pose>0 0 0 0 0 0</pose>
+	</link>
+	<joint type="fixed" name="base_link_to_chassis">
+		<child link="chassis_link"/>
+		<parent link="base_link"/>
+	</joint>
+	<!-- Define the chassis of the differential drive robot, which is our base -->
+	<link name='chassis_link'>
+		<!-- Define inertial system for the chassis -->
+		<inertial>
+			<mass value="${m_chassis}"/>
+			<xacro:box_inertia m="${m_chassis}" x="${x_chassis}" y="${y_chassis}" z="${z_chassis}"/>
+		</inertial>
+		<!-- Define collision sorrounding box -->
+		<collision name='collision'>
+			<origin xyz="0 0 0" rpy=" 0 0 0"/>
+			<geometry>
+				<box size="${x_chassis} ${y_chassis} ${z_chassis}"/>
+			</geometry>
+		</collision>
+		<!-- Define visualization structure -->
+		<visual name='base_link_visual'>
+			<origin xyz="0 0 0" rpy=" 0 0 0"/>
+			<geometry>
+				<box size="${x_chassis} ${y_chassis} ${z_chassis}"/>
+			</geometry>
+			<material name="yellow"/>
+		</visual>
+		<!-- RPY and batt block -->
+		<collision name='batt_rpy_collision'>
+			<origin xyz="${-0.03} 0 ${0.02+z_chassis/2}" rpy=" 0 0 0"/>
+			<geometry>
+				<box size="${0.12} ${0.1} ${0.04}" />
+			</geometry>
+			<surface>
+				<friction>
+					<ode>
+						<mu>0</mu>
+						<mu2>0</mu2>
+						<slip1>1.0</slip1>
+						<slip2>1.0</slip2>
+					</ode>
+				</friction>
+			</surface>
+		</collision>
+		<visual name='batt_rpy_visual'>
+			<origin xyz="${-0.03} 0 ${0.02+z_chassis/2}" rpy=" 0 0 0"/>
+			<geometry>
+				<box size="${0.12} ${0.1} ${0.04}" />
+			</geometry>
+			<material name="red">
+				<color rgba="0.80078125 0.12890625 0.1328125 1.0"/>
+			</material>
+		</visual>
+		<!-- Add the caster wheel! Here we simply assume complete slippage, thus we do not require that it rotates! -->
+		<collision name='caster_collision'>
+			<origin xyz="${-(r_wheel/2)+x_chassis/2} 0 ${-r_wheel/2-z_chassis/2}" rpy=" 0 0 0"/>
+			<geometry>
+				<sphere radius="${r_wheel/2}"/>
+			</geometry>
+			<surface>
+				<friction>
+					<ode>
+						<mu>0</mu>
+						<mu2>0</mu2>
+						<slip1>1.0</slip1>
+						<slip2>1.0</slip2>
+					</ode>
+				</friction>
+			</surface>
+		</collision>
+		<visual name='caster_visual'>
+			<origin xyz="${-(r_wheel/2)+x_chassis/2} 0 ${-r_wheel/2-z_chassis/2}" rpy=" 0 0 0"/>
+			<geometry>
+				<sphere radius="${r_wheel/2}"/>
+			</geometry>
+			<material name="black"/>
+		</visual>
+	</link>
+	<!-- Radar -->
+	<link name="radar">
+		<visual>
+			<geometry>
+				<box size="${x_radar} ${y_radar} ${z_radar}" />
+			</geometry>
+			<material name="red"/>
+		</visual>
+	</link>
+	<joint type="fixed" name="base_link_to_radar">
+		<origin xyz="${0.04+x_radar/2} 0 ${z_radar/2+z_chassis/2}" rpy="0 0 0"/>
+		<child link="radar"/>
+		<parent link="base_link"/>
+	</joint>
+	<!-- Add the wheels for the robot -->
+	<link name="left_wheel">
+		<collision name="collision">
+			<origin xyz="0 0 0" rpy="0 1.5707 1.5707"/>
+			<geometry>
+				<cylinder radius="${r_wheel}" length="${h_wheel}"/>
+			</geometry>
+			<surface>
+				<friction>
+					<ode>
+						<mu>1.0</mu>
+						<mu2>1.0</mu2>
+						<slip1>0.0</slip1>
+						<slip2>0.0</slip2>
+					</ode>
+				</friction>
+			</surface>
+		</collision>
+		<visual name="left_wheel_visual">
+			<origin xyz="0 0 0" rpy="0 1.5707 1.5707"/>
+			<geometry>
+				<cylinder radius="${r_wheel}" length="${h_wheel}"/>
+			</geometry>
+			<material name="black"/>
+		</visual>
+		<inertial>
+			<origin xyz="0 0 0" rpy="0 1.5707 1.5707"/>
+			<mass value="${m_wheel}"/>
+			<cylinder_inertia m="${m_wheel}" r="${r_wheel}" h="${h_wheel}"/>
+			<xacro:cylinder_inertia m="${m_wheel}" r="${r_wheel}" h="${h_wheel}"/>
+		</inertial>
+	</link>
+	<link name="right_wheel">
+		<collision name="collision">
+			<origin xyz="0 0 0" rpy="0 1.5707 1.5707"/>
+			<geometry>
+				<cylinder radius="${r_wheel}" length="${h_wheel}"/>
+			</geometry>
+			<surface>
+				<friction>
+					<ode>
+						<mu>1.0</mu>
+						<mu2>1.0</mu2>
+						<slip1>0.0</slip1>
+						<slip2>0.0</slip2>
+					</ode>
+				</friction>
+			</surface>
+		</collision>
+		<visual name="right_wheel_visual">
+			<origin xyz="0 0 0" rpy="0 1.5707 1.5707"/>
+			<geometry>
+				<cylinder radius="${r_wheel}" length="${h_wheel}"/>
+			</geometry>
+			<material name="black"/>
+		</visual>
+		<inertial>
+			<origin xyz="0 0 0" rpy="0 1.5707 1.5707"/>
+			<mass value="${m_wheel}"/>
+			<cylinder_inertia m="${m_wheel}" r="${r_wheel}" h="${h_wheel}"/>
+			<xacro:cylinder_inertia m="${m_wheel}" r="${r_wheel}" h="${h_wheel}"/>
+		</inertial>
+	</link>
+	<!-- Set joints for the wheels which can be controlled over ROS -->
+	<joint type="continuous" name="left_wheel_hinge">
+		<origin xyz="${-x_chassis/4} ${y_chassis/2+h_wheel/2} ${-z_chassis/2}" rpy="0 0 0"/>
+		<child link="left_wheel"/>
+		<parent link="base_link"/>
+		<axis xyz="0 1 0" rpy="0 0 0"/>
+		<limit effort="100" velocity="100"/>
+		<joint_properties damping="0.0" friction="0.0"/>
+	</joint>
+	<joint type="continuous" name="right_wheel_hinge">
+		<origin xyz="${-x_chassis/4} ${-y_chassis/2-h_wheel/2} ${-z_chassis/2}" rpy="0 0 0"/>
+		<child link="right_wheel"/>
+		<parent link="base_link"/>
+		<axis xyz="0 1 0" rpy="0 0 0"/>
+		<limit effort="100" velocity="100"/>
+		<joint_properties damping="0.0" friction="0.0"/>
+	</joint>
 </robot>

File: src/dviratis_robotas/urdf/parameter.xacro (robot description, xacro)
@@ -3,6 +3,6 @@
     <!-- Define parameter for the differential drive robot -->
     <!-- Parameter for the chassis, size [m] and mass [kg] -->
-    <xacro:property name="x_chassis" value="0.23" />
-    <xacro:property name="y_chassis" value="0.12" />
+    <xacro:property name="x_chassis" value="0.27" />
+    <xacro:property name="y_chassis" value="0.15" />
     <xacro:property name="z_chassis" value="0.01" />
     <xacro:property name="m_chassis" value="1.0" />
@@ -17,7 +17,7 @@
     <xacro:property name="h_camera" value="0.1" />
     <!-- Radar parameters -->
-    <xacro:property name="x_radar" value="0.1" />
-    <xacro:property name="y_radar" value="0.1" />
-    <xacro:property name="z_radar" value="0.1" />
+    <xacro:property name="x_radar" value="0.01" />
+    <xacro:property name="y_radar" value="0.065" />
+    <xacro:property name="z_radar" value="0.085" />
     <!-- Parameters for the Hukoyu Laser -->
     <xacro:property name="x_hokuyo" value="0.1" />

Commit message: Kamera, lazeris su pluginu

File: src/dviratis_robotas/urdf/dr_robotas.xacro (robot description, xacro)
@@ -40,7 +40,7 @@
 		<!-- RPY and batt block -->
 		<collision name='batt_rpy_collision'>
-			<origin xyz="${-0.03} 0 ${0.02+z_chassis/2}" rpy=" 0 0 0"/>
-			<geometry>
-				<box size="${0.12} ${0.1} ${0.04}" />
+			<origin xyz="${offset_rpybat} 0 ${z_rpybat/2+z_chassis/2}" rpy=" 0 0 0"/>
+			<geometry>
+				<box size="${x_rpybat} ${y_rpybat} ${z_rpybat}" />
 			</geometry>
 			<surface>
@@ -56,7 +56,7 @@
 		</collision>
 		<visual name='batt_rpy_visual'>
-			<origin xyz="${-0.03} 0 ${0.02+z_chassis/2}" rpy=" 0 0 0"/>
-			<geometry>
-				<box size="${0.12} ${0.1} ${0.04}" />
+			<origin xyz="${offset_rpybat} 0 ${z_rpybat/2+z_chassis/2}" rpy=" 0 0 0"/>
+			<geometry>
+				<box size="${x_rpybat} ${y_rpybat} ${z_rpybat}" />
 			</geometry>
 			<material name="red">
@@ -97,8 +97,46 @@
 			<material name="red"/>
 		</visual>
+		<collision>
+			<geometry>
+				<box size="${x_radar} ${y_radar} ${z_radar}" />
+			</geometry>
+		</collision>
 	</link>
 	<joint type="fixed" name="base_link_to_radar">
-		<origin xyz="${0.04+x_radar/2} 0 ${z_radar/2+z_chassis/2}" rpy="0 0 0"/>
+		<origin xyz="${0.015+x_radar/2+x_rpybat/2+offset_rpybat} 0 ${z_radar/2+z_chassis/2}" rpy="0 0 0"/>
 		<child link="radar"/>
+		<parent link="base_link"/>
+	</joint>
+	<!-- Camera -->
+	<link name="camera">
+		<!-- lens -->
+		<visual name="cam_lens_visual">
+			<geometry>
+				<cylinder radius="${r_camera}" length="${h_camera}"/>
+			</geometry>
+			<material name="grey"/>
+		</visual>
+		<collision name="cam_lens_collision">
+			<geometry>
+				<cylinder radius="${r_camera}" length="${h_camera}"/>
+			</geometry>
+		</collision>
+		<!-- chassis -->
+		<visual name="cam_chassis_visual">
+			<origin xyz="0 0 ${-h_camera/2+h_camera/6}" rpy="0 0 0"/>
+			<geometry>
+				<box size="${xy_cam_chassis} ${xy_cam_chassis} ${h_camera/3}" />
+			</geometry>
+			<material name="grey"/>
+		</visual>
+		<collision name="cam_chassis_collision">
+			<geometry>
+				<box size="${xy_cam_chassis} ${xy_cam_chassis} ${h_camera/3}" />
+			</geometry>
+		</collision>
+	</link>
+	<joint type="fixed" name="base_link_to_cam">
+		<origin xyz="${h_camera/2+0.015*2+x_radar+(x_rpybat/2+offset_rpybat)} 0 ${xy_cam_chassis/2+z_chassis/2}" rpy="0 1.5707 0"/>
+		<child link="camera"/>
 		<parent link="base_link"/>
 	</joint>

File: src/dviratis_robotas/urdf/parameter.xacro (robot description, xacro)
@@ -3,8 +3,13 @@
     <!-- Define parameter for the differential drive robot -->
     <!-- Parameter for the chassis, size [m] and mass [kg] -->
-    <xacro:property name="x_chassis" value="0.27" />
-    <xacro:property name="y_chassis" value="0.15" />
+    <xacro:property name="x_chassis" value="0.22" />
+    <xacro:property name="y_chassis" value="0.12" />
     <xacro:property name="z_chassis" value="0.01" />
     <xacro:property name="m_chassis" value="1.0" />
+    <!-- RPY and battery -->
+    <xacro:property name="x_rpybat" value="0.12" />
+    <xacro:property name="y_rpybat" value="0.1" />
+    <xacro:property name="z_rpybat" value="0.04" />
+    <xacro:property name="offset_rpybat" value="-0.01" />
     <!-- Parameter for the wheels, radius [m], height [m], mass [kg], torque [Nm], wheelbase [m] -->
     <xacro:property name="r_wheel" value="0.035"/>
@@ -14,13 +19,10 @@
     <xacro:property name="L_wheel" value="0.00" />
     <!-- Camera parameters -->
-    <xacro:property name="r_camera" value="0.1" />
-    <xacro:property name="h_camera" value="0.1" />
+    <xacro:property name="r_camera" value="0.01" />
+    <xacro:property name="h_camera" value="0.03" />
+    <xacro:property name="xy_cam_chassis" value="0.04" />
     <!-- Radar parameters -->
     <xacro:property name="x_radar" value="0.01" />
     <xacro:property name="y_radar" value="0.065" />
     <xacro:property name="z_radar" value="0.085" />
-    <!-- Parameters for the Hukoyu Laser -->
-    <xacro:property name="x_hokuyo" value="0.1" />
-    <xacro:property name="y_hokuyo" value="0.1" />
-    <xacro:property name="z_hokuyo" value="0.1" />
 </robot>

Commit message: Kameros upgrade

File: src/dviratis_robotas/urdf/dr_robotas.xacro (robot description, xacro)
@@ -92,4 +92,5 @@
 	<link name="radar">
 		<visual>
+			<origin xyz="0 0 ${-z_radar/4}" rpy="0 0 0"/>
 			<geometry>
 				<box size="${x_radar} ${y_radar} ${z_radar}" />
@@ -104,12 +105,13 @@
 	</link>
 	<joint type="fixed" name="base_link_to_radar">
-		<origin xyz="${0.015+x_radar/2+x_rpybat/2+offset_rpybat} 0 ${z_radar/2+z_chassis/2}" rpy="0 0 0"/>
+		<origin xyz="${0.015+x_radar/2+x_rpybat/2+offset_rpybat} 0 ${z_radar/2+z_chassis/2+z_radar/4}" rpy="0 0 0"/>
 		<child link="radar"/>
 		<parent link="base_link"/>
 	</joint>
 	<!-- Camera -->
-	<link name="camera">
+	<link name="camera_link">
 		<!-- lens -->
 		<visual name="cam_lens_visual">
+			<origin xyz="0 0 0" rpy="0 1.5707 0"/>
 			<geometry>
 				<cylinder radius="${r_camera}" length="${h_camera}"/>
@@ -118,4 +120,5 @@
 		</visual>
 		<collision name="cam_lens_collision">
+			<origin xyz="0 0 0" rpy="0 1.5707 0"/>
 			<geometry>
 				<cylinder radius="${r_camera}" length="${h_camera}"/>
@@ -124,19 +127,19 @@
 		<!-- chassis -->
 		<visual name="cam_chassis_visual">
-			<origin xyz="0 0 ${-h_camera/2+h_camera/6}" rpy="0 0 0"/>
+			<origin xyz="${-h_camera/2+h_camera/4} 0 0" rpy="0 0 0"/>
+			<geometry>
+				<box size="${h_camera/2} ${xy_cam_chassis} ${xy_cam_chassis}" />
+			</geometry>
+			<material name="grey"/>
+		</visual>
+		<collision name="cam_chassis_collision">
 			<geometry>
 				<box size="${xy_cam_chassis} ${xy_cam_chassis} ${h_camera/3}" />
 			</geometry>
-			<material name="grey"/>
-		</visual>
-		<collision name="cam_chassis_collision">
-			<geometry>
-				<box size="${xy_cam_chassis} ${xy_cam_chassis} ${h_camera/3}" />
-			</geometry>
 		</collision>
 	</link>
 	<joint type="fixed" name="base_link_to_cam">
-		<origin xyz="${h_camera/2+0.015*2+x_radar+(x_rpybat/2+offset_rpybat)} 0 ${xy_cam_chassis/2+z_chassis/2}" rpy="0 1.5707 0"/>
-		<child link="camera"/>
+		<origin xyz="${h_camera/2+0.015*2+x_radar+(x_rpybat/2+offset_rpybat)} 0 ${xy_cam_chassis/2+z_chassis/2}" rpy="0 0 0"/>
+		<child link="camera_link"/>
 		<parent link="base_link"/>
 	</joint>

Commit message: Modelio papildymai

File: src/dviratis_robotas/urdf/dr_robotas.xacro (robot description, xacro)
@@ -144,4 +144,22 @@
 		<parent link="base_link"/>
 	</joint>
+	<link name="pcb_link">
+		<visual name="pcb_link_visual">
+			<geometry>
+				<box size="${x_pcb} ${y_pcb} ${z_pcb}" />
+			</geometry>
+			<material name="green"/>
+		</visual>
+		<collision name="pcb_link_collision">
+			<geometry>
+				<box size="${x_pcb} ${y_pcb} ${z_pcb}" />
+			</geometry>
+		</collision>
+	</link>
+	<joint type="fixed" name="base_link_to_pcb">
+		<origin xyz="${-(x_pcb/2+x_rpybat/2-offset_rpybat+0.01)} 0 ${z_pcb/2+z_chassis/2}" rpy="0 0 0"/>
+		<child link="pcb_link"/>
+		<parent link="base_link"/>
+	</joint>
 	<!-- Add the wheels for the robot -->
 	<link name="left_wheel">

File: src/dviratis_robotas/urdf/parameter.xacro (robot description, xacro)
@@ -3,6 +3,6 @@
     <!-- Define parameter for the differential drive robot -->
     <!-- Parameter for the chassis, size [m] and mass [kg] -->
-    <xacro:property name="x_chassis" value="0.22" />
-    <xacro:property name="y_chassis" value="0.12" />
+    <xacro:property name="x_chassis" value="0.24" />
+    <xacro:property name="y_chassis" value="0.14" />
     <xacro:property name="z_chassis" value="0.01" />
     <xacro:property name="m_chassis" value="1.0" />
@@ -11,5 +11,5 @@
     <xacro:property name="y_rpybat" value="0.1" />
     <xacro:property name="z_rpybat" value="0.04" />
-    <xacro:property name="offset_rpybat" value="-0.01" />
+    <xacro:property name="offset_rpybat" value="-0.00" />
     <!-- Parameter for the wheels, radius [m], height [m], mass [kg], torque [Nm], wheelbase [m] -->
     <xacro:property name="r_wheel" value="0.035"/>
@@ -26,3 +26,7 @@
     <xacro:property name="y_radar" value="0.065" />
     <xacro:property name="z_radar" value="0.085" />
+    <!-- PCB -->
+    <xacro:property name="x_pcb" value="0.04" />
+    <xacro:property name="y_pcb" value="0.06" />
+    <xacro:property name="z_pcb" value="0.005" />
 </robot>
