Commit message: Pries testus su kitais modeliais

File: src/dviratis_robotas/urdf/dr_robotas.xacro (robot description, xacro)
@@ -169,14 +169,4 @@
 				<cylinder radius="${r_wheel}" length="${h_wheel}"/>
 			</geometry>
-			<surface>
-				<friction>
-					<ode>
-						<mu>1.0</mu>
-						<mu2>1.0</mu2>
-						<slip1>0.0</slip1>
-						<slip2>0.0</slip2>
-					</ode>
-				</friction>
-			</surface>
 		</collision>
 		<visual name="left_wheel_visual">
@@ -200,14 +190,4 @@
 				<cylinder radius="${r_wheel}" length="${h_wheel}"/>
 			</geometry>
-			<surface>
-				<friction>
-					<ode>
-						<mu>1.0</mu>
-						<mu2>1.0</mu2>
-						<slip1>0.0</slip1>
-						<slip2>0.0</slip2>
-					</ode>
-				</friction>
-			</surface>
 		</collision>
 		<visual name="right_wheel_visual">
@@ -231,6 +211,6 @@
 		<parent link="base_link"/>
 		<axis xyz="0 1 0" rpy="0 0 0"/>
-		<limit effort="100" velocity="100"/>
-		<joint_properties damping="0.0" friction="0.0"/>
+		<limit effort="10000" velocity="1000"/>
+		<joint_properties damping="1.0" friction="1.0"/>
 	</joint>
 	<joint type="continuous" name="right_wheel_hinge">
@@ -239,6 +219,6 @@
 		<parent link="base_link"/>
 		<axis xyz="0 1 0" rpy="0 0 0"/>
-		<limit effort="100" velocity="100"/>
-		<joint_properties damping="0.0" friction="0.0"/>
+		<limit effort="10000" velocity="1000"/>
+		<joint_properties damping="1.0" friction="1.0"/>
 	</joint>
 </robot>

File: src/dviratis_robotas/urdf/parameter.xacro (robot description, xacro)
@@ -6,5 +6,5 @@
     <xacro:property name="y_chassis" value="0.14" />
     <xacro:property name="z_chassis" value="0.01" />
-    <xacro:property name="m_chassis" value="1.0" />
+    <xacro:property name="m_chassis" value="0.5" />
     <!-- RPY and battery -->
     <xacro:property name="x_rpybat" value="0.12" />

Commit message: vaziuoja normaliai su kitu urdf

File: src/dviratis_robotas/urdf/dr_robotas.xacro (robot description, xacro)
@@ -1,224 +1,81 @@
-<?xml version='1.0'?>
-<!-- choose a name space and start xacro -->
+<?xml version="1.0" ?>
 <robot name="dr_robotas"
-	xmlns:xacro="http://www.ros.org/wiki/xacro">
-	<!-- Start by including all required xacro files which hold the macros -->
-	<xacro:include filename="$(find dviratis_robotas)/urdf/diff_drive.gazebo" />
-	<xacro:include filename="$(find dviratis_robotas)/urdf/materials.xacro" />
-	<xacro:include filename="$(find dviratis_robotas)/urdf/macros.xacro" />
-	<xacro:include filename="$(find dviratis_robotas)/urdf/parameter.xacro" />
-	<!-- Create a dummy link as base link -->
-	<link name='base_link'>
-		<pose>0 0 0 0 0 0</pose>
-	</link>
-	<joint type="fixed" name="base_link_to_chassis">
-		<child link="chassis_link"/>
-		<parent link="base_link"/>
-	</joint>
-	<!-- Define the chassis of the differential drive robot, which is our base -->
-	<link name='chassis_link'>
-		<!-- Define inertial system for the chassis -->
-		<inertial>
-			<mass value="${m_chassis}"/>
-			<xacro:box_inertia m="${m_chassis}" x="${x_chassis}" y="${y_chassis}" z="${z_chassis}"/>
-		</inertial>
-		<!-- Define collision sorrounding box -->
-		<collision name='collision'>
-			<origin xyz="0 0 0" rpy=" 0 0 0"/>
-			<geometry>
-				<box size="${x_chassis} ${y_chassis} ${z_chassis}"/>
-			</geometry>
-		</collision>
-		<!-- Define visualization structure -->
-		<visual name='base_link_visual'>
-			<origin xyz="0 0 0" rpy=" 0 0 0"/>
-			<geometry>
-				<box size="${x_chassis} ${y_chassis} ${z_chassis}"/>
-			</geometry>
-			<material name="yellow"/>
-		</visual>
-		<!-- RPY and batt block -->
-		<collision name='batt_rpy_collision'>
-			<origin xyz="${offset_rpybat} 0 ${z_rpybat/2+z_chassis/2}" rpy=" 0 0 0"/>
-			<geometry>
-				<box size="${x_rpybat} ${y_rpybat} ${z_rpybat}" />
-			</geometry>
-			<surface>
-				<friction>
-					<ode>
-						<mu>0</mu>
-						<mu2>0</mu2>
-						<slip1>1.0</slip1>
-						<slip2>1.0</slip2>
-					</ode>
-				</friction>
-			</surface>
-		</collision>
-		<visual name='batt_rpy_visual'>
-			<origin xyz="${offset_rpybat} 0 ${z_rpybat/2+z_chassis/2}" rpy=" 0 0 0"/>
-			<geometry>
-				<box size="${x_rpybat} ${y_rpybat} ${z_rpybat}" />
-			</geometry>
-			<material name="red">
-				<color rgba="0.80078125 0.12890625 0.1328125 1.0"/>
-			</material>
-		</visual>
-		<!-- Add the caster wheel! Here we simply assume complete slippage, thus we do not require that it rotates! -->
-		<collision name='caster_collision'>
-			<origin xyz="${-(r_wheel/2)+x_chassis/2} 0 ${-r_wheel/2-z_chassis/2}" rpy=" 0 0 0"/>
-			<geometry>
-				<sphere radius="${r_wheel/2}"/>
-			</geometry>
-			<surface>
-				<friction>
-					<ode>
-						<mu>0</mu>
-						<mu2>0</mu2>
-						<slip1>1.0</slip1>
-						<slip2>1.0</slip2>
-					</ode>
-				</friction>
-			</surface>
-		</collision>
-		<visual name='caster_visual'>
-			<origin xyz="${-(r_wheel/2)+x_chassis/2} 0 ${-r_wheel/2-z_chassis/2}" rpy=" 0 0 0"/>
-			<geometry>
-				<sphere radius="${r_wheel/2}"/>
-			</geometry>
-			<material name="black"/>
-		</visual>
-	</link>
-	<!-- Radar -->
-	<link name="radar">
-		<visual>
-			<origin xyz="0 0 ${-z_radar/4}" rpy="0 0 0"/>
-			<geometry>
-				<box size="${x_radar} ${y_radar} ${z_radar}" />
-			</geometry>
-			<material name="red"/>
-		</visual>
-		<collision>
-			<geometry>
-				<box size="${x_radar} ${y_radar} ${z_radar}" />
-			</geometry>
-		</collision>
-	</link>
-	<joint type="fixed" name="base_link_to_radar">
-		<origin xyz="${0.015+x_radar/2+x_rpybat/2+offset_rpybat} 0 ${z_radar/2+z_chassis/2+z_radar/4}" rpy="0 0 0"/>
-		<child link="radar"/>
-		<parent link="base_link"/>
-	</joint>
-	<!-- Camera -->
-	<link name="camera_link">
-		<!-- lens -->
-		<visual name="cam_lens_visual">
-			<origin xyz="0 0 0" rpy="0 1.5707 0"/>
-			<geometry>
-				<cylinder radius="${r_camera}" length="${h_camera}"/>
-			</geometry>
-			<material name="grey"/>
-		</visual>
-		<collision name="cam_lens_collision">
-			<origin xyz="0 0 0" rpy="0 1.5707 0"/>
-			<geometry>
-				<cylinder radius="${r_camera}" length="${h_camera}"/>
-			</geometry>
-		</collision>
-		<!-- chassis -->
-		<visual name="cam_chassis_visual">
-			<origin xyz="${-h_camera/2+h_camera/4} 0 0" rpy="0 0 0"/>
-			<geometry>
-				<box size="${h_camera/2} ${xy_cam_chassis} ${xy_cam_chassis}" />
-			</geometry>
-			<material name="grey"/>
-		</visual>
-		<collision name="cam_chassis_collision">
-			<geometry>
-				<box size="${xy_cam_chassis} ${xy_cam_chassis} ${h_camera/3}" />
-			</geometry>
-		</collision>
-	</link>
-	<joint type="fixed" name="base_link_to_cam">
-		<origin xyz="${h_camera/2+0.015*2+x_radar+(x_rpybat/2+offset_rpybat)} 0 ${xy_cam_chassis/2+z_chassis/2}" rpy="0 0 0"/>
-		<child link="camera_link"/>
-		<parent link="base_link"/>
-	</joint>
-	<link name="pcb_link">
-		<visual name="pcb_link_visual">
-			<geometry>
-				<box size="${x_pcb} ${y_pcb} ${z_pcb}" />
-			</geometry>
-			<material name="green"/>
-		</visual>
-		<collision name="pcb_link_collision">
-			<geometry>
-				<box size="${x_pcb} ${y_pcb} ${z_pcb}" />
-			</geometry>
-		</collision>
-	</link>
-	<joint type="fixed" name="base_link_to_pcb">
-		<origin xyz="${-(x_pcb/2+x_rpybat/2-offset_rpybat+0.01)} 0 ${z_pcb/2+z_chassis/2}" rpy="0 0 0"/>
-		<child link="pcb_link"/>
-		<parent link="base_link"/>
-	</joint>
-	<!-- Add the wheels for the robot -->
-	<link name="left_wheel">
-		<collision name="collision">
-			<origin xyz="0 0 0" rpy="0 1.5707 1.5707"/>
-			<geometry>
-				<cylinder radius="${r_wheel}" length="${h_wheel}"/>
-			</geometry>
-		</collision>
-		<visual name="left_wheel_visual">
-			<origin xyz="0 0 0" rpy="0 1.5707 1.5707"/>
-			<geometry>
-				<cylinder radius="${r_wheel}" length="${h_wheel}"/>
-			</geometry>
-			<material name="black"/>
-		</visual>
-		<inertial>
-			<origin xyz="0 0 0" rpy="0 1.5707 1.5707"/>
-			<mass value="${m_wheel}"/>
-			<cylinder_inertia m="${m_wheel}" r="${r_wheel}" h="${h_wheel}"/>
-			<xacro:cylinder_inertia m="${m_wheel}" r="${r_wheel}" h="${h_wheel}"/>
-		</inertial>
-	</link>
-	<link name="right_wheel">
-		<collision name="collision">
-			<origin xyz="0 0 0" rpy="0 1.5707 1.5707"/>
-			<geometry>
-				<cylinder radius="${r_wheel}" length="${h_wheel}"/>
-			</geometry>
-		</collision>
-		<visual name="right_wheel_visual">
-			<origin xyz="0 0 0" rpy="0 1.5707 1.5707"/>
-			<geometry>
-				<cylinder radius="${r_wheel}" length="${h_wheel}"/>
-			</geometry>
-			<material name="black"/>
-		</visual>
-		<inertial>
-			<origin xyz="0 0 0" rpy="0 1.5707 1.5707"/>
-			<mass value="${m_wheel}"/>
-			<cylinder_inertia m="${m_wheel}" r="${r_wheel}" h="${h_wheel}"/>
-			<xacro:cylinder_inertia m="${m_wheel}" r="${r_wheel}" h="${h_wheel}"/>
-		</inertial>
-	</link>
-	<!-- Set joints for the wheels which can be controlled over ROS -->
-	<joint type="continuous" name="left_wheel_hinge">
-		<origin xyz="${-x_chassis/4} ${y_chassis/2+h_wheel/2} ${-z_chassis/2}" rpy="0 0 0"/>
-		<child link="left_wheel"/>
-		<parent link="base_link"/>
-		<axis xyz="0 1 0" rpy="0 0 0"/>
-		<limit effort="10000" velocity="1000"/>
-		<joint_properties damping="1.0" friction="1.0"/>
-	</joint>
-	<joint type="continuous" name="right_wheel_hinge">
-		<origin xyz="${-x_chassis/4} ${-y_chassis/2-h_wheel/2} ${-z_chassis/2}" rpy="0 0 0"/>
-		<child link="right_wheel"/>
-		<parent link="base_link"/>
-		<axis xyz="0 1 0" rpy="0 0 0"/>
-		<limit effort="10000" velocity="1000"/>
-		<joint_properties damping="1.0" friction="1.0"/>
-	</joint>
+    xmlns:xacro="http://www.ros.org/wiki/xacro">
+    <xacro:include filename="$(find dviratis_robotas)/urdf/materials.xacro" />
+    <xacro:include filename="$(find dviratis_robotas)/urdf/dr_robotas.gazebo" />
+    <xacro:include filename="$(find dviratis_robotas)/urdf/macros.xacro" />
+    <link name="link_chassis">
+        <!-- pose and inertial -->
+        <pose>0 0 0.1 0 0 0</pose>
+        <inertial>
+            <mass value="5"/>
+            <origin rpy="0 0 0" xyz="0 0 0.1"/>
+            <inertia ixx="0.0395416666667" ixy="0" ixz="0" iyy="0.106208333333" iyz="0" izz="0.106208333333"/>
+        </inertial>
+        <!-- body -->
+        <collision name="collision_chassis">
+            <geometry>
+                <box size="0.5 0.3 0.07"/>
+            </geometry>
+        </collision>
+        <visual>
+            <origin rpy="0 0 0" xyz="0 0 0"/>
+            <geometry>
+                <box size="0.5 0.3 0.07"/>
+            </geometry>
+            <material name="blue"/>
+        </visual>
+        <!-- caster front -->
+        <collision name="caster_front_collision">
+            <origin rpy=" 0 0 0" xyz="0.35 0 -0.05"/>
+            <geometry>
+                <sphere radius="0.05"/>
+            </geometry>
+            <surface>
+                <friction>
+                    <ode>
+                        <mu>0</mu>
+                        <mu2>0</mu2>
+                        <slip1>1.0</slip1>
+                        <slip2>1.0</slip2>
+                    </ode>
+                </friction>
+            </surface>
+        </collision>
+        <visual name="caster_front_visual">
+            <origin rpy=" 0 0 0" xyz="0.2 0 -0.05"/>
+            <geometry>
+                <sphere radius="0.05"/>
+            </geometry>
+        </visual>
+    </link>
+    <link name="sensor_laser">
+        <inertial>
+            <origin xyz="0 0 0" rpy="0 0 0" />
+            <mass value="1" />
+            <xacro:cylinder_inertia mass="1" r="0.05" l="0.1" />
+        </inertial>
+        <visual>
+            <origin xyz="0 0 0" rpy="0 0 0" />
+            <geometry>
+                <cylinder radius="0.05" length="0.1"/>
+            </geometry>
+            <material name="white" />
+        </visual>
+        <collision>
+            <origin xyz="0 0 0" rpy="0 0 0"/>
+            <geometry>
+                <cylinder radius="0.05" length="0.1"/>
+            </geometry>
+        </collision>
+    </link>
+    <joint name="joint_sensor_laser" type="fixed">
+        <origin xyz="0.15 0 0.05" rpy="0 0 0"/>
+        <parent link="link_chassis"/>
+        <child link="sensor_laser"/>
+    </joint>
+    <xacro:link_wheel name="link_right_wheel" />
+    <xacro:joint_wheel name="joint_right_wheel" child="link_right_wheel" origin_xyz="-0.05 0.20 0" />
+    <xacro:link_wheel name="link_left_wheel" />
+    <xacro:joint_wheel name="joint_left_wheel" child="link_left_wheel" origin_xyz="-0.05 -0.20 0" />
 </robot>

File: src/dviratis_robotas/urdf/macros.xacro (robot description, xacro)
@@ -1,9 +1,37 @@
 <?xml version="1.0"?>
-<robot xmlns:xacro="http://www.ros.org/wiki/xacro">
-    <xacro:macro name="box_inertia" params="m x y z">
-        <inertia ixx="${m*(y*y+z*z)/12}" ixy = "0" ixz = "0" iyy="${m*(x*x+z*z)/12}" iyz = "0" izz="${m*(x*x+z*z)/12}" />
+<robot xmlns:xacro="http://wiki.ros.org/xacro">
+    <xacro:macro name="link_wheel" params="name">
+        <link name="${name}">
+            <inertial>
+                <mass value="0.2"/>
+                <origin rpy="0 1.5707 1.5707" xyz="0 0 0"/>
+                <inertia ixx="0.000526666666667" ixy="0" ixz="0" iyy="0.000526666666667" iyz="0" izz="0.001"/>
+            </inertial>
+            <collision name="link_right_wheel_collision">
+                <origin rpy="0 1.5707 1.5707" xyz="0 0 0"/>
+                <geometry>
+                    <cylinder length="0.04" radius="0.1"/>
+                </geometry>
+            </collision>
+            <visual name="${name}_visual">
+                <origin rpy="0 1.5707 1.5707" xyz="0 0 0"/>
+                <geometry>
+                    <cylinder length="0.04" radius="0.1"/>
+                </geometry>
+            </visual>
+        </link>
     </xacro:macro>
-    <xacro:macro name="cylinder_inertia" params="m r h">
-        <inertia ixx="${m*(3*r*r+h*h)/12}" ixy = "0" ixz = "0" iyy="${m*(3*r*r+h*h)/12}" iyz = "0" izz="${m*r*r/2}" />
+    <xacro:macro name="joint_wheel" params="name child origin_xyz">
+        <joint name="${name}" type="continuous">
+            <origin rpy="0 0 0" xyz="${origin_xyz}"/>
+            <child link="${child}"/>
+            <parent link="link_chassis"/>
+            <axis rpy="0 0 0" xyz="0 1 0"/>
+            <limit effort="10000" velocity="1000"/>
+            <joint_properties damping="1.0" friction="1.0"/>
+        </joint>
+    </xacro:macro>
+    <xacro:macro name="cylinder_inertia" params="mass r l">
+        <inertia ixx="${mass*(3*r*r+l*l)/12}" ixy = "0" ixz = "0" iyy="${mass*(3*r*r+l*l)/12}" iyz = "0" izz="${mass*(r*r)/2}" />
     </xacro:macro>
 </robot>

File: src/dviratis_robotas/urdf1/materials.xacro (robot description, xacro)
@@ -1,4 +1,7 @@
-<?xml version="1.0" ?>
-<robot xmlns:xacro="http://wiki.ros.org/xacro">
+<?xml version="1.0"?>
+<robot xmlns:xacro="http://www.ros.org/wiki/xacro">
+    <material name="orange">
+        <color rgba="${255/255} ${108/255} ${10/255} 1.0"/>
+    </material>
     <material name="black">
         <color rgba="0.0 0.0 0.0 1.0"/>
@@ -13,7 +16,4 @@
         <color rgba="0.2 0.2 0.2 1.0"/>
     </material>
-    <material name="orange">
-        <color rgba="1.0 0.423529411765 0.0392156862745 1.0"/>
-    </material>
     <material name="brown">
         <color rgba="0.870588235294 0.811764705882 0.764705882353 1.0"/>
@@ -25,3 +25,6 @@
         <color rgba="1.0 1.0 1.0 1.0"/>
     </material>
+    <material name="yellow">
+        <color rgba="1.0 1.0 0 1.0"/>
+    </material>
 </robot>
